File: LoudMouth.kicad_pcb (KiCad board)
At the start: 2 copper layers, 27.4 x 32 mm, 15 parts, among them P101 CONN_01X02, P102 CONN_01X02, P103 CONN_01X02, Q101 Q_NPN_BCE

Commit message: Finished Class A board, ready to send to fab
Parts:
- added REF**: MountingHole_2-5mm, Mounting_Holes:MountingHole_2-5mm, F.Cu at (180.5, 121.0)
- added REF**: MountingHole_2-5mm, Mounting_Holes:MountingHole_2-5mm, F.Cu at (159.0, 120.9)
- added REF**: MountingHole_2-5mm, Mounting_Holes:MountingHole_2-5mm, F.Cu at (158.9, 94.9)
- added REF**: MountingHole_2-5mm, Mounting_Holes:MountingHole_2-5mm, F.Cu at (180.4, 94.7)
- added TP101: CONN_01X01, Measurement_Points:Measurement_Point_Round-SMD-Pad_Big, F.Cu at (163.8, 121.6)
- added TP102: CONN_01X01, Measurement_Points:Measurement_Point_Round-SMD-Pad_Big, F.Cu at (163.6, 94.4)
- added TP103: CONN_01X01, Measurement_Points:Measurement_Point_Round-SMD-Pad_Big, F.Cu at (176.0, 97.8)
- Q101: value Q_NPN_BCE -> Q_NPN_EBC
- moved P101 11.0 mm to (158.6, 109.5), turned to 180 degrees
- moved P102 10.1 mm to (168.3, 94.1), turned to 90 degrees
- moved R102 4.19 mm to (165.8, 114.6)
- moved Q101 2.81 mm to (170.2, 111.0), turned to 90 degrees
- moved C101 1.25 mm to (160.1, 113.8), turned to 180 degrees
Connections:
- P101 pad 1: GND -> /IN
- P101 pad 2: /IN -> GND
- Q101 pad 1: Net-(Q101-Pad1) -> /EMITTER
- Q101 pad 2: Net-(Q101-Pad2) -> /BASE
- Q101 pad 3: Net-(Q101-Pad3) -> /COLLECTOR
- R103 pad 1: Net-(Q101-Pad1) -> /BASE
- R105 pad 1: Net-(Q101-Pad2) -> /COLLECTOR
- R106 pad 2: Net-(Q101-Pad3) -> /EMITTER
Routing:
- net /IN: track 4.81 -> 15.7 mm
- net GND: track 23.6 -> 12.8 mm, vias 1 -> 3
- net /OUT: track 7.53 -> 14.1 mm
- net /BASE: track 0.00 -> 4.67 mm
- net Net-(Q101-Pad1): track 4.54 -> 0.00 mm
- net Net-(Q101-Pad2): track 4.32 -> 0.00 mm
- net Net-(C101-Pad1): track 9.17 -> 12.6 mm
- net /COLLECTOR: track 0.00 -> 3.39 mm
- net /EMITTER: track 0.00 -> 3.30 mm
- net Net-(Q101-Pad3): track 3.06 -> 0.00 mm
Other:
- board text added: "B"
- board text added: "C"
- board text added: "E"
- board text added: "IN"
- board text added: "OUT"
- board text added: "VCC"
