File: ClassD/hw/_autosave-ClassD.kicad_pcb (KiCad board)
At the start: 2 copper layers, 81.2 x 56.9 mm, 310 parts, among them P1 RedRCA, P2 WhiteRCA, P3 CONN_01X02, P4 CONN_01X02, P5 CONN_01X02, SW1 SW_PUSH, SW2 SW_PUSH, U1 TDA7491LP, U2 MCP1700T

Commit message: Finished layout with DRC
Routing:
- net /VCC: track 99.5 -> 100.1 mm
Changed lines of the file:
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@@
   (general
     (links 372)
-    (no_connects 281)
+    (no_connects 0)
     (area 121.961839 87.255279 203.275001 144.301281)
     (thickness 1.6)
@@
   (page A4)
   (layers
-    (0 F.Cu signal)
+    (0 F.Cu signal hide)
     (31 B.Cu signal)
     (32 B.Adhes user)
@@
   (segment (start 160.31464 113.16208) (end 159.62884 113.84788) (width 0.3048) (layer B.Cu) (net 18))
   (segment (start 202.17384 95.72498) (end 202.17384 116.03228) (width 0.6096) (layer B.Cu) (net 19))
-  (segment (start 195.98894 88.37168) (end 197.34784 89.73058) (width 0.6096) (layer B.Cu) (net 19))
-  (segment (start 197.34784 89.73058) (end 197.34784 91.35618) (width 0.6096) (layer B.Cu) (net 19))
-  (segment (start 197.34784 91.35618) (end 198.77024 92.77858) (width 0.6096) (layer B.Cu) (net 19))
-  (segment (start 198.77024 92.77858) (end 200.90384 92.77858) (width 0.6096) (layer B.Cu) (net 19))
-  (segment (start 200.90384 92.77858) (end 202.17384 94.04858) (width 0.6096) (layer B.Cu) (net 19))
+  (segment (start 195.98894 88.37168) (end 196.83984 89.22258) (width 0.6096) (layer B.Cu) (net 19))
+  (segment (start 196.83984 89.22258) (end 196.83984 91.99118) (width 0.6096) (layer B.Cu) (net 19))
+  (segment (start 196.83984 91.99118) (end 198.38924 93.54058) (width 0.6096) (layer B.Cu) (net 19))
+  (segment (start 198.38924 93.54058) (end 201.66584 93.54058) (width 0.6096) (layer B.Cu) (net 19))
+  (segment (start 201.66584 93.54058) (end 202.17384 94.04858) (width 0.6096) (layer B.Cu) (net 19))
   (segment (start 202.17384 94.04858) (end 202.17384 95.72498) (width 0.6096) (layer B.Cu) (net 19))
   (segment (start 161.55924 88.37168) (end 195.98894 88.37168) (width 0.6096) (layer B.Cu) (net 19))
@@
     (connect_pads yes (clearance 0.254))
     (min_thickness 0.254)
-    (fill (arc_segments 16) (thermal_gap 0.508) (thermal_bridge_width 0.508))
+    (fill yes (arc_segments 16) (thermal_gap 0.508) (thermal_bridge_width 0.508))
     (polygon
       (pts
@@
     (connect_pads yes (clearance 0.508))
     (min_thickness 0.254)
-    (fill (arc_segments 16) (thermal_gap 0.508) (thermal_bridge_width 0.508))
+    (fill yes (arc_segments 16) (thermal_gap 0.508) (thermal_bridge_width 0.508))
     (polygon
       (pts
@@
     (connect_pads yes (clearance 0.508))
     (min_thickness 0.254)
-    (fill (arc_segments 16) (thermal_gap 0.508) (thermal_bridge_width 0.508))
+    (fill yes (arc_segments 16) (thermal_gap 0.508) (thermal_bridge_width 0.508))
     (polygon
       (pts
@@
     (connect_pads yes (clearance 0.254))
     (min_thickness 0.254)
-    (fill (arc_segments 16) (thermal_gap 0.508) (thermal_bridge_width 0.508))
+    (fill yes (arc_segments 16) (thermal_gap 0.508) (thermal_bridge_width 0.508))
     (polygon
       (pts
@@
     (connect_pads yes (clearance 0.254))
     (min_thickness 0.254)
-    (fill (arc_segments 16) (thermal_gap 0.508) (thermal_bridge_width 0.508))
+    (fill yes (arc_segments 16) (thermal_gap 0.508) (thermal_bridge_width 0.508))
     (polygon
       (pts
